Commit message: [bebop] Fix prefix for links and joints. Add fdm_ports as parameters

File: models/bebop/urdf/bebop.urdf.xacro (robot description, xacro)
@@ -3,5 +3,7 @@
   <xacro:property name="enable_velodyne" value="$(arg enable_velodyne)"/>
 	<xacro:property name="enable_magnet" value="$(arg enable_magnet)"/>
-  <xacro:property name="namespace" value="$(arg namespace)" />
+  	<xacro:property name="namespace" value="$(arg namespace)" />
+  	<xacro:property name="fdm_port_in" value="$(arg fdm_port_in)"/>
+	<xacro:property name="fdm_port_out" value="$(arg fdm_port_out)"/>
   <!-- Instantiate bebop "mechanics" -->
 	<xacro:include filename="$(find ardupilot_gazebo)/models/bebop/urdf/bebop_base.urdf.xacro" />
@@ -11,5 +13,5 @@
 		namespace="${namespace}"
 		odometry_sensor_suffix=""
-		parent_link="base_link"
+		parent_link="${namespace}/base_link"
 		pose_topic="pose"
 		pose_with_covariance_topic="pose_with_covariance"
@@ -41,5 +43,5 @@
 		namespace="${namespace}"
 		odometry_sensor_suffix="gt"
-		parent_link="base_link"
+		parent_link="${namespace}/base_link"
 		pose_topic="pose_gt"
 		pose_with_covariance_topic="pose_with_covariance_gt"
@@ -68,14 +70,14 @@
 	</xacro:odometry_plugin_macro>
 	<xacro:ardupilot
-		imu_topic="/bebop/imu"
-		control_topic="/bebop/gazebo/command/motor_speed"
-		imu_sensor_name="bebop::imu_link::imu_sensor"
-		rotor_0_joint="bebop::rotor_0_joint"
-		rotor_1_joint="bebop::rotor_1_joint"
-		rotor_2_joint="bebop::rotor_2_joint"
-		rotor_3_joint="bebop::rotor_3_joint"
+		imu_topic="${namespace}/imu"
+		control_topic="${namespace}/gazebo/command/motor_speed"
+		imu_sensor_name="${namespace}::imu_link::imu_sensor"
+		rotor_0_joint="${namespace}::${namespace}/rotor_0_joint"
+		rotor_1_joint="${namespace}::${namespace}/rotor_1_joint"
+		rotor_2_joint="${namespace}::${namespace}/rotor_2_joint"
+		rotor_3_joint="${namespace}::${namespace}/rotor_3_joint"
 		thrust_multiplier="1000"
-		fdm_port_in="9002"
-		fdm_port_out="9003">
+		fdm_port_in="${fdm_port_in}"
+		fdm_port_out="${fdm_port_out}">
 	</xacro:ardupilot>
     <link name="laser1D_link">
@@ -89,5 +91,5 @@
       <!--<axis xyz="0 0 1" />-->
       <origin xyz="0.111 0 0.0217" rpy="0 0 0"/>
-      <parent link="base_link"/>
+      <parent link="$(arg namespace)/base_link"/>
       <child link="laser1D_link"/>
     </joint>
@@ -161,5 +163,5 @@
 	<gazebo>
 		<plugin name="dipole_magnet" filename="libstorm_gazebo_dipole_magnet.so">
-			<bodyName>bebop::base_link</bodyName>
+			<bodyName>${namespace}::base_link</bodyName>
 			<dipole_moment>0 0 50</dipole_moment>
 			<!-- Set to false if not using ROS -->

File: models/bebop/urdf/bebop_base.urdf.xacro (robot description, xacro)
@@ -57,5 +57,5 @@
     motor_constant="${motor_constant}"
     moment_constant="${moment_constant}"
-    parent="base_link"
+    parent="$(arg namespace)/base_link"
     mass_rotor="${mass_rotor}"
     radius_rotor="${radius_rotor}"
@@ -77,5 +77,5 @@
     motor_constant="${motor_constant}"
     moment_constant="${moment_constant}"
-    parent="base_link"
+    parent="$(arg namespace)/base_link"
     mass_rotor="${mass_rotor}"
     radius_rotor="${radius_rotor}"
@@ -97,5 +97,5 @@
     motor_constant="${motor_constant}"
     moment_constant="${moment_constant}"
-    parent="base_link"
+    parent="$(arg namespace)/base_link"
     mass_rotor="${mass_rotor}"
     radius_rotor="${radius_rotor}"
@@ -117,5 +117,5 @@
     motor_constant="${motor_constant}"
     moment_constant="${moment_constant}"
-    parent="base_link"
+    parent="$(arg namespace)/base_link"
     mass_rotor="${mass_rotor}"
     radius_rotor="${radius_rotor}"
@@ -148,5 +148,5 @@
     camera_link="${camera_link}"
     camera_mass="${camera_mass}"
-    parent="base_link">
+    parent="$(arg namespace)/base_link">
     <!-- Front Facing Camera -->
     <!--origin xyz="0.111 0 0.0217" rpy="0 1.57079632 0"/-->
