Commit message: Added initial gimbal model to simulation

File: models/kopterworx/urdf/kopterworx.urdf.xacro (robot description, xacro)
@@ -3,9 +3,10 @@
   <xacro:property name="namespace" value="$(arg namespace)" />
   <xacro:property name="enable_velodyne" value="$(arg enable_velodyne)"/>
-	<xacro:property name="enable_rotating_velodyne" value="$(arg enable_rotating_velodyne)" />
-	<xacro:property name="fdm_port_in" value="$(arg fdm_port_in)"/>
-	<xacro:property name="fdm_port_out" value="$(arg fdm_port_out)"/>
-	<xacro:property name="max_range" value="$(arg max_range)"/>
-	<gazebo>
+  <xacro:property name="enable_gimbal" value="$(arg enable_gimbal)"/>
+  <xacro:property name="enable_rotating_velodyne" value="$(arg enable_rotating_velodyne)"/>
+  <xacro:property name="fdm_port_in" value="$(arg fdm_port_in)"/>
+  <xacro:property name="fdm_port_out" value="$(arg fdm_port_out)"/>
+  <xacro:property name="max_range" value="$(arg max_range)"/>
+  <gazebo>
     <plugin name="gazebo_ros_control" filename="libgazebo_ros_control.so">
       <robotNamespace>/$(arg namespace)</robotNamespace>
@@ -14,13 +15,13 @@
     </plugin>
   </gazebo>
-	<xacro:property name="horizontal_velodyne_origin">
+  <xacro:property name="horizontal_velodyne_origin">
     <origin xyz="0.08 0. -0.1578" rpy="-3.141592653589793 0.1323284641020683 0." />
-	</xacro:property>
-	<xacro:property name="front_facing_camera">
-		<origin xyz="0.2 0 0.05" rpy="0 0 0"/>
-	</xacro:property>
-	<xacro:property name="down_facing_camera">
+  </xacro:property>
+  <xacro:property name="front_facing_camera">
+	<origin xyz="0.2 0 0.05" rpy="0 0 0"/>
+  </xacro:property>
+  <xacro:property name="down_facing_camera">
 	  <origin xyz="0 0.2 -0.3" rpy="-1.570796 1.570796 0"/>
-	</xacro:property>
+  </xacro:property>
   <xacro:property name="camera_mass" value="1e-5"/>
 	<xacro:property name="camera_size" value="0.05" />
@@ -33,22 +34,25 @@
   </xacro:property>
   <!-- Instantiate kopterworx mechanics "mechanics" -->
-	<xacro:include filename="$(find ardupilot_gazebo)/models/kopterworx/urdf/kopterworx_base.urdf.xacro" />
+  <xacro:include filename="$(find ardupilot_gazebo)/models/kopterworx/urdf/kopterworx_base.urdf.xacro" />
   <xacro:include filename="$(find rotors_description)/urdf/component_snippets.xacro" />
-	<!-- Ardupilot plugin -->
+  <!-- Add xacro model of a gimbal -->
+  <!--xacro:include filename="$(find ardupilot_gazebo)/models/utils/.." -->
+  <xacro:include filename="$(find ardupilot_gazebo)/models/util/gimbal.urdf.xacro" />
+  <!-- Ardupilot plugin -->
   <xacro:ardupilot
-		imu_topic="/${namespace}/imu"
-		control_topic="/${namespace}/gazebo/command/motor_speed"
-		imu_sensor_name="${namespace}::imu_link::imu_sensor"
-		rotor_0_joint="${namespace}::${namespace}/rotor_0_joint"
-		rotor_1_joint="${namespace}::${namespace}/rotor_1_joint"
-		rotor_2_joint="${namespace}::${namespace}/rotor_2_joint"
-		rotor_3_joint="${namespace}::${namespace}/rotor_3_joint"
-		thrust_multiplier="600"
-		fdm_port_in="${fdm_port_in}"
-		fdm_port_out="${fdm_port_out}">
-	</xacro:ardupilot>
-	<xacro:if value="${enable_velodyne}">
-		<xacro:if value="${enable_rotating_velodyne}">
-			<xacro:include filename="$(find velodyne_description)/urdf/LiDAR-X-rotating.urdf.xacro"/>
+    imu_topic="/${namespace}/imu"
+	control_topic="/${namespace}/gazebo/command/motor_speed"
+	imu_sensor_name="${namespace}::imu_link::imu_sensor"
+	rotor_0_joint="${namespace}::${namespace}/rotor_0_joint"
+	rotor_1_joint="${namespace}::${namespace}/rotor_1_joint"
+	rotor_2_joint="${namespace}::${namespace}/rotor_2_joint"
+	rotor_3_joint="${namespace}::${namespace}/rotor_3_joint"
+	thrust_multiplier="600"
+	fdm_port_in="${fdm_port_in}"
+	fdm_port_out="${fdm_port_out}">
+  </xacro:ardupilot>
+  <xacro:if value="${enable_velodyne}">
+	<xacro:if value="${enable_rotating_velodyne}">
+		<xacro:include filename="$(find velodyne_description)/urdf/LiDAR-X-rotating.urdf.xacro"/>
 			<xacro:lidar-x
 				parent="${namespace}/base_link_inertia"
@@ -63,7 +67,7 @@
 				<xacro:insert_block name="horizontal_velodyne_origin"/>
 			</xacro:lidar-x>
-		</xacro:if>
-		<xacro:unless value="${enable_rotating_velodyne}">
-			<xacro:include filename="$(find velodyne_description)/urdf/LiDAR-X.urdf.xacro"/>
+	</xacro:if>
+	<xacro:unless value="${enable_rotating_velodyne}">
+		<xacro:include filename="$(find velodyne_description)/urdf/LiDAR-X.urdf.xacro"/>
 			<xacro:lidar-x
 				parent="${namespace}/base_link_inertia"
@@ -79,5 +83,5 @@
 			</xacro:lidar-x>
 		</xacro:unless>
-	</xacro:if>
+  </xacro:if>
 	<!-- Realistic odometry sensor with noise -->
 	<xacro:odometry_plugin_macro
@@ -111,14 +115,18 @@
 	</xacro:odometry_plugin_macro>
 <!-- Choose one of the following (and comment out the other): fixed RGBD camera or gimbal with RGBD camera. -->
-  <xacro:cam
-    namespace="$(arg namespace)"
-    camera_link="${camera_size}"
-    camera_mass="${camera_mass}"
-    parent="${namespace}/base_link">
-		<xacro:insert_block name="front_facing_camera"/>
+    <xacro:cam
+      namespace="$(arg namespace)"
+      camera_link="${camera_size}"
+      camera_mass="${camera_mass}"
+      parent="${namespace}/base_link">
+	<xacro:insert_block name="front_facing_camera"/>
     <xacro:insert_block name="camera_inertia"/>
-  </xacro:cam>
-<!--   <xacro:gimbal_macro parent="base_link">
-    <origin xyz="0.25 0 -0.1" rpy="0 0 0"/>
-  </xacro:gimbal_macro> -->
+    </xacro:cam>
+  	<xacro:if value="$(arg enable_gimbal)">
+		<xacro:gimbal
+			parent="${namespace}/base_link"
+			xyz="0.0 0.0 0.0"
+			rpy="0.0 0.0 0.0">
+		</xacro:gimbal>
+  	</xacro:if>
 </robot>

Commit message: [kopterworx] Add enable_gimbal option

File: models/kopterworx/urdf/kopterworx.urdf.xacro (robot description, xacro)
@@ -9,4 +9,5 @@
 	<xacro:property name="max_range" value="$(arg max_range)"/>
 	<xacro:property name="laser_count" value="$(arg laser_count)"/>
+	<xacro:property name="enable_gimbal" value="$(arg enable_gimbal)"/>
 	<gazebo>
     <plugin name="gazebo_ros_control" filename="libgazebo_ros_control.so">
@@ -127,17 +128,20 @@
 		<origin xyz="0.0 0.0 0.0" rpy="0.0 0.0 0.0" />
 	</xacro:odometry_plugin_macro>
-<!-- Choose one of the following (and comment out the other): fixed RGBD camera or gimbal with RGBD camera. -->
-  <xacro:cam
-    namespace="$(arg namespace)"
-    camera_link="${camera_size}"
-    camera_mass="${camera_mass}"
-    parent="${namespace}/base_link">
-		<xacro:insert_block name="front_facing_camera"/>
-    <xacro:insert_block name="camera_inertia"/>
-  </xacro:cam>
-	<!-- <xacro:gimbal_macro
-		namespace="$(arg namespace)"
-		parent="${namespace}/base_link">
-	<origin xyz="0.25 0 -0.1" rpy="0 0 0"/>
-	</xacro:gimbal_macro> -->
+	<xacro:if value="${enable_gimbal}">
+		<xacro:gimbal_macro
+			namespace="$(arg namespace)"
+			parent="${namespace}/base_link">
+		<origin xyz="0.25 0 -0.1" rpy="0 0 0"/>
+		</xacro:gimbal_macro>
+	</xacro:if>
+	<xacro:unless value="${enable_gimbal}">
+		<xacro:cam
+			namespace="$(arg namespace)"
+			camera_link="${camera_size}"
+			camera_mass="${camera_mass}"
+			parent="${namespace}/base_link">
+				<xacro:insert_block name="front_facing_camera"/>
+			<xacro:insert_block name="camera_inertia"/>
+		</xacro:cam>
+	</xacro:unless>
 </robot>

Commit message: Mesh file from parent xacro

File: models/kopterworx/urdf/kopterworx.urdf.xacro (robot description, xacro)
@@ -35,4 +35,5 @@
     ixy="0.0" ixz="0.0" iyz="0.0" />
   </xacro:property>
+	<xacro:property name="mesh_file" value="ardupilot_gazebo/models/kopterworx/meshes/kopterworx_model_simple.dae" />
   <!-- Instantiate kopterworx mechanics "mechanics" -->
 	<xacro:include filename="$(find ardupilot_gazebo)/models/kopterworx/urdf/kopterworx_base.urdf.xacro" />

File: models/kopterworx/urdf/kopterworx_base.urdf.xacro (robot description, xacro)
@@ -6,5 +6,4 @@
   <!-- Body Properties -->
   <xacro:property name="rotor_velocity_slowdown_sim" value="15" />
-  <xacro:property name="mesh_file" value="ardupilot_gazebo/models/kopterworx/meshes/kopterworx_model_simple.dae" />
   <xacro:property name="mesh_scale" value="0.1" />
   <xacro:property name="prop_scale" value="0.002" />
