Commit message: Reverse camera pose

File: models/kopterworx/urdf/kopterworx_falcon.urdf.xacro (robot description, xacro)
@@ -136,5 +136,5 @@
 			namespace="$(arg namespace)"
 			parent="${namespace}/base_link">
-		<origin xyz="-0.25 0 -0.1" rpy="0 0 3.14"/>
+		<origin xyz="0.25 0 -0.1" rpy="0 0 0"/>
 		</xacro:gimbal_macro>
 	</xacro:if>
